Commit message: Add A* planner, AMCL localization, MPC controller, and benchmark harness
Grow the ROS 2 stack from Pure-Pursuit-on-a-fixed-path to a full
plan -> localize -> control -> benchmark pipeline in the maze.

Planning (new vto_planning):
- A* grid planner (framework-free astar.py): 8-connectivity, octile heuristic,
  clearance-aware cost (keeps paths corridor-centered) and hard C-space inflation
  by the robot radius. astar_planner_node publishes nav_msgs/Path.
- generate_maze.py also emits a map_server occupancy map (maze.pgm/yaml) from the
  same wall geometry; resolution 0.1 m.

Localization (Phase 2):
- Add a 2D lidar to the robot; nav2 map_server + AMCL own a live map->odom.
- Refactor the planner and Pure Pursuit to the map frame via TF (map->base),
  replacing the static "poor-man's localization" transform so AMCL actually
  corrects odometry drift (verified over a ~100 m drive).

Control (vto_control):
- Pure Pursuit upgraded: adaptive lookahead, turn-in-place at sharp corners, and
  curvature slowdown, split into a framework-free pursuit_core. Fixes corner
  collisions, a bootstrap stall, and a sparse-path carrot spin.
- MPC controller: nonlinear receding-horizon control (CasADi + IPOPT), unicycle
  model, tracking/effort/comfort/terminal costs, multiple shooting (mpc_core).
  Drop-in with Pure Pursuit via controller:=pursuit|mpc.

Benchmark (new vto_bench):
- Goal-tour harness measuring 7 metrics (cross-track, time, len-ratio, comfort,
  effort, clearance, compute) per leg, deterministic seeded tour, per-leg CSV +
  tour poses. Both controllers publish /controller/compute_ms.

Robot / infra:
- Blue robot, rear caster (4-point base, less accel slip), lidar sensor.
- Dockerfile installs casadi.
- Docs 07-14 (planner, QoS/frames, integration, C-space+following, AMCL,
  map-frame refactor, MPC, benchmarking) + trajectory-optimization report.

Co-Authored-By: Claude Opus 4.8 <noreply@anthropic.com>

File: ros2_ws/src/vto_description/urdf/mobile/diffbot.gazebo.xacro (robot description, xacro)
@@ -15,6 +15,36 @@
     <mu1>1.0</mu1> <mu2>1.0</mu2>
   </gazebo>
-  <gazebo reference="caster">
+  <gazebo reference="front_caster">
     <mu1>0.0</mu1> <mu2>0.0</mu2>
   </gazebo>
+  <gazebo reference="rear_caster">
+    <mu1>0.0</mu1> <mu2>0.0</mu2>
+  </gazebo>
+  <!-- 2D lidar: gz publishes gz.msgs.LaserScan on gz topic /scan (bridged to ROS
+       /scan). gz_frame_id=laser so the scan's frame matches the URDF TF frame.
+       Needs the gz-sim-sensors-system plugin in the world (maze.sdf has it). -->
+  <gazebo reference="laser">
+    <sensor name="lidar" type="gpu_lidar">
+      <topic>scan</topic>
+      <update_rate>10</update_rate>
+      <always_on>1</always_on>
+      <visualize>true</visualize>
+      <gz_frame_id>laser</gz_frame_id>
+      <lidar>
+        <scan>
+          <horizontal>
+            <samples>360</samples>
+            <resolution>1</resolution>
+            <min_angle>-3.141592</min_angle>
+            <max_angle>3.141592</max_angle>
+          </horizontal>
+        </scan>
+        <range>
+          <min>0.15</min>
+          <max>12.0</max>
+          <resolution>0.01</resolution>
+        </range>
+      </lidar>
+    </sensor>
+  </gazebo>
 </robot>

File: ros2_ws/src/vto_description/urdf/mobile/diffbot.urdf.xacro (robot description, xacro)
@@ -35,5 +35,5 @@
     <visual>
       <geometry><box size="${base_len} ${base_wid} ${base_hei}"/></geometry>
-      <material name="steel"><color rgba="0.4 0.45 0.5 1"/></material>
+      <material name="robot_blue"><color rgba="0.1 0.35 0.85 1"/></material>
     </visual>
     <collision>
@@ -70,17 +70,38 @@
   <xacro:wheel prefix="left"  side_y="${ wheel_separation/2}"/>
   <xacro:wheel prefix="right" side_y="${-wheel_separation/2}"/>
-  <!-- ================= caster (passive) ================= -->
-  <link name="caster">
-    <visual><geometry><sphere radius="${wheel_radius*0.6}"/></geometry></visual>
-    <collision><geometry><sphere radius="${wheel_radius*0.6}"/></geometry></collision>
-    <xacro:cyl_inertia m="0.2" r="${wheel_radius*0.6}" l="0.02"/>
-  </link>
-  <joint name="caster_joint" type="fixed">
-    <parent link="base_link"/>
-    <child  link="caster"/>
-    <origin xyz="${base_len/2 - wheel_radius} 0 ${-wheel_zoff - wheel_radius*0.4}"/>
-  </joint>
+  <!-- ================= casters (passive, fore & aft) =================
+       Two ball casters symmetric about the drive-wheel axis (x=0) give a 4-point
+       base (2 drive wheels + 2 casters) so the body doesn't pitch under accel;
+       steadier normal load on the drive wheels -> less load-transfer slip. -->
+  <xacro:macro name="caster" params="prefix x">
+    <link name="${prefix}_caster">
+      <visual><geometry><sphere radius="${wheel_radius*0.6}"/></geometry></visual>
+      <collision><geometry><sphere radius="${wheel_radius*0.6}"/></geometry></collision>
+      <xacro:cyl_inertia m="0.2" r="${wheel_radius*0.6}" l="0.02"/>
+    </link>
+    <joint name="${prefix}_caster_joint" type="fixed">
+      <parent link="base_link"/>
+      <child  link="${prefix}_caster"/>
+      <origin xyz="${x} 0 ${-wheel_zoff - wheel_radius*0.4}"/>
+    </joint>
+  </xacro:macro>
+  <xacro:caster prefix="front" x="${  base_len/2 - wheel_radius}"/>
+  <xacro:caster prefix="rear"  x="${-(base_len/2 - wheel_radius)}"/>
   <!-- ================= ros2_control + Gazebo ================= -->
   <xacro:include filename="$(find vto_description)/urdf/mobile/diffbot.ros2_control.xacro"/>
+  <!-- ================= 2D lidar (Phase 2: AMCL localization) ================= -->
+  <link name="laser">
+    <visual>
+      <geometry><cylinder radius="0.035" length="0.04"/></geometry>
+      <material name="lidar_black"><color rgba="0.1 0.1 0.1 1"/></material>
+    </visual>
+    <collision><geometry><cylinder radius="0.035" length="0.04"/></geometry></collision>
+    <xacro:cyl_inertia m="0.1" r="0.035" l="0.04"/>
+  </link>
+  <joint name="laser_joint" type="fixed">
+    <parent link="base_link"/>
+    <child  link="laser"/>
+    <origin xyz="${base_len/2 - 0.06} 0 ${base_hei/2 + 0.02}"/>
+  </joint>
   <xacro:include filename="$(find vto_description)/urdf/mobile/diffbot.gazebo.xacro"/>
 </robot>

Commit message: Add Ackermann robot stack: description/control/EKF/AMCL, lattice+Dubins+Reeds-Shepp planning, acados MPC, Follower planner, rooms maze, and diffdrive doc updates
Builds out the full car-like (M2) pipeline alongside the existing diffbot
one: ackermannbot URDF/ros2_control/Gazebo bringup, TF-based pure pursuit
and acados SQP MPC controllers, a state-lattice planner over a Dubins
primitive library (with heading-index and clearance-penalty cost fixes),
a Reeds-Shepp reverse-motion solver (built, verified, not yet wired into
the live planner), a 5-room maze variant that sidesteps a proven
forward-only reachability gap, and the Follower planner (A* guidance +
PID/dynamic-bicycle-model trajectory generation, ported from src/GP,
verified live in Gazebo). Also extends the benchmark harness for
Ackermann tours and adds diffdrive EKF/DWA/nav-pipeline docs.

Docs 16-41 and 47-48 cover the full design rationale, method-selection
trade-offs, and interview-angle notes for each step.

Co-Authored-By: Claude Sonnet 5 <noreply@anthropic.com>

File: ros2_ws/src/vto_description/urdf/mobile/diffbot.gazebo.xacro (robot description, xacro)
@@ -48,3 +48,32 @@
     </sensor>
   </gazebo>
+  <!-- IMU: gz publishes gz.msgs.IMU on gz topic /imu (bridged to ROS /imu).
+       gz_frame_id=imu_link so orientation/angular_velocity/linear_acceleration
+       are expressed in the IMU's own frame (REP-145). Needs the
+       gz-sim-imu-system plugin in the world (separate from the lidar's
+       gz-sim-sensors-system — IMU is not a rendering-based sensor).
+       Gaussian noise (typical low-cost MEMS gyro/accel figures) is required,
+       not cosmetic: it's what makes gz populate non-zero covariance on the
+       message, which ekf_node's Kalman gain needs — zero covariance reads as
+       "infinitely certain" and breaks/short-circuits the fusion math. -->
+  <gazebo reference="imu_link">
+    <sensor name="imu" type="imu">
+      <topic>imu</topic>
+      <update_rate>100</update_rate>
+      <always_on>1</always_on>
+      <gz_frame_id>imu_link</gz_frame_id>
+      <imu>
+        <angular_velocity>
+          <x><noise type="gaussian"><mean>0.0</mean><stddev>2e-4</stddev></noise></x>
+          <y><noise type="gaussian"><mean>0.0</mean><stddev>2e-4</stddev></noise></y>
+          <z><noise type="gaussian"><mean>0.0</mean><stddev>2e-4</stddev></noise></z>
+        </angular_velocity>
+        <linear_acceleration>
+          <x><noise type="gaussian"><mean>0.0</mean><stddev>1.7e-2</stddev></noise></x>
+          <y><noise type="gaussian"><mean>0.0</mean><stddev>1.7e-2</stddev></noise></y>
+          <z><noise type="gaussian"><mean>0.0</mean><stddev>1.7e-2</stddev></noise></z>
+        </linear_acceleration>
+      </imu>
+    </sensor>
+  </gazebo>
 </robot>

File: ros2_ws/src/vto_description/urdf/mobile/diffbot.urdf.xacro (robot description, xacro)
@@ -104,4 +104,16 @@
     <origin xyz="${base_len/2 - 0.06} 0 ${base_hei/2 + 0.02}"/>
   </joint>
+  <!-- ================= IMU (Phase 2: robot_localization EKF) =================
+       Placed at base_link's own origin (not offset like the lidar) so
+       linear_acceleration reflects true body acceleration rather than a
+       lever-arm/centripetal term picked up from sitting off-center in turns. -->
+  <link name="imu_link">
+    <xacro:box_inertia m="0.05" x="0.02" y="0.02" z="0.02"/>
+  </link>
+  <joint name="imu_joint" type="fixed">
+    <parent link="base_link"/>
+    <child  link="imu_link"/>
+    <origin xyz="0 0 0"/>
+  </joint>
   <xacro:include filename="$(find vto_description)/urdf/mobile/diffbot.gazebo.xacro"/>
 </robot>
